File: PCB/chordsense_afe/chordsense_afe.kicad_sch (KiCad schematic)
At the start: 25 parts, among them IC1 MCP6002-I_P, IC2 MCP6002-I_P, J1 ACJS-MHDR, J2 ACJS-MHDR, J3 Conn_01x08, J4 SJ3-35053B, U2 MCP3201

Commit message: initial PCB finished, ready to order remaining parts
Parts:
- J4: footprint SJ3-35053B:SAMESKY_SJ3-35053B -> Connector_PinHeader_2.54mm:PinHeader_1x04_P2.54mm_Vertical
- VR1: footprint PDB182-K425K-103A:Bourns-PDB182-K425K-103A-0 -> Connector_PinHeader_2.54mm:PinHeader_1x06_P2.54mm_Vertical
Changed lines of the file:
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@@
 			)
 		)
-		(property "Footprint" "PDB182-K425K-103A:Bourns-PDB182-K425K-103A-0"
+		(property "Footprint" "Connector_PinHeader_2.54mm:PinHeader_1x06_P2.54mm_Vertical"
 			(at 76.2 127 0)
 			(hide yes)
@@
 			)
 		)
-		(property "Footprint" "PDB182-K425K-103A:Bourns-PDB182-K425K-103A-0"
+		(property "Footprint" "Connector_PinHeader_2.54mm:PinHeader_1x06_P2.54mm_Vertical"
 			(at 76.2 162.56 0)
 			(hide yes)
@@
 			)
 		)
-		(property "Footprint" "SJ3-35053B:SAMESKY_SJ3-35053B"
+		(property "Footprint" "Connector_PinHeader_2.54mm:PinHeader_1x04_P2.54mm_Vertical"
 			(at 227.33 129.54 0)
 			(hide yes)

Commit message: pcb fixes (wider holds for acjs)
Parts:
- removed J3: Conn_01x08, Connector_PinHeader_2.54mm:PinHeader_1x08_P2.54mm_Vertical, symbol Connector_Generic:Conn_01x08
- added J5, J6: Conn_01x04, Connector_JST:JST_XH_B4B-XH-A_1x04_P2.50mm_Vertical, symbol Connector_Generic:Conn_01x04
- J4: footprint Connector_PinHeader_2.54mm:PinHeader_1x04_P2.54mm_Vertical -> Connector_JST:JST_XH_B4B-XH-A_1x04_P2.50mm_Vertical
- VR1: footprint Connector_PinHeader_2.54mm:PinHeader_1x06_P2.54mm_Vertical -> Connector_JST:JST_XH_B6B-XH-A_1x06_P2.50mm_Vertical
Connections:
- net +3.3V: now also J5.1 (Pin_1)
- net GND: now also J1.2, J2.2, J6.4 (Pin_4); no longer J1.4, J2.4
- net PI_BCK: now also J5.4 (Pin_4)
- net PI_CLK: now also J6.1 (Pin_1)
- net PI_CS: now also J6.3 (Pin_3)
- net PI_Din: now also J5.3 (Pin_3)
- net PI_Dout: now also J6.2 (Pin_2)
- net PI_wsel: now also J5.2 (Pin_2)
- net at C1.1, R2.1: now also J1.1, J2.1; no longer J1.3, J2.3
